File: kicad/a-register.sch (KiCad schematic (older format))
At the start: 2 parts

Commit message: Final Commit Pre-Talk The final commit before Monday's talk, including the PDF of the schematic to make it accessible.
Parts:
- gave numbers to parts that had none: 2
Other:
- note added: "The 74HC541 is the line buffer, which has its inputs connected to the"
- note added: "The 74HC547 is the set of 8 D-type flip flops, with its inputs connected"
- note added: "always outputs and the clock signal is hooked up to AI."
- note added: "enable lines are connected to the control signal AO."
- note added: "registers internal bus and its outputs connected to the data bus. Its output"
- note added: "to the data bus and its outputs to an internal bus which goes\n"
- note added: "to the line buffer and the adder. Its output enable pin is tied such that it"
- moved on the sheet: U1, U2
