File: kicad/adder.sch (KiCad schematic (older format))
At the start: 3 parts

Commit message: Final Commit Pre-Talk The final commit before Monday's talk, including the PDF of the schematic to make it accessible.
Parts:
- gave numbers to parts that had none: 3
Other:
- note added: "The adder gets constant input from the A and B registers, and"
- note added: "act as 1 8-bit adder."
- note added: "constantly outputs its result to the line buffer chip (similarly to the"
- note added: "full adders, one of which outputs a carry bit to the other, allowing them to"
- note added: "registers), which only asserts to the data bus when the EO control"
- note added: "signal is asserted. The actual adding is done by 2 74HC283 4-bit binary"
- moved on the sheet: U5, U6, U7
