File: kicad/b-register.sch (KiCad schematic (older format))
At the start: 2 parts

Commit message: Final Commit Pre-Talk The final commit before Monday's talk, including the PDF of the schematic to make it accessible.
Parts:
- gave numbers to parts that had none: 2
Other:
- note added: "The only difference between the A and B registers is that the B registers"
- note added: "internal bus is connected to the variable storage's address bus as well as"
- note added: "to the adder."
- moved on the sheet: U3, U4
