File: kicad/comparison-unit.sch (KiCad schematic (older format))
At the start: 4 parts

Commit message: Final Commit Pre-Talk The final commit before Monday's talk, including the PDF of the schematic to make it accessible.
Parts:
- gave numbers to parts that had none: 4
Other:
- note added: "74HC85s to act as a single 8-bit comparator. The two 74HC573A"
- note added: "The comparators output their result to the instruction decoder where it is"
- note added: "The comparison unit consists of two data latches (chips that can 'latch'"
- note added: "comparators which, similarly to the adders and counters elsewhere in"
- note added: "latches are used to store the two words to compare, each one storing"
- note added: "the CPU have outputs that can carry between chips, allowing the two"
- note added: "the current value of a bus and output it) being fed into two 4-bit"
- note added: "the value of the data bus on the relevant control signal of either L1 or L2."
- note added: "used as part of the instruction lookup process."
- moved on the sheet: U10, U11, U8, U9
