File: kicad/data-bus-termination.sch (KiCad schematic (older format))
At the start: 8 parts

Commit message: Final Commit Pre-Talk The final commit before Monday's talk, including the PDF of the schematic to make it accessible.
Parts:
- gave numbers to parts that had none: 8
Other:
- note added: "This sheet only exists because the logic chips used don't like it when an"
- note added: "input isn't specifically high or low, so this termination makes it so that if"
- note added: "nothing is asserted to the data bus, a low value will be asserted."
- moved on the sheet: R1, R2, R3, R4, R5, R6, R7, R8
