File: kicad/instruction-decoder.sch (KiCad schematic (older format))
At the start: 3 parts

Commit message: Final Commit Pre-Talk The final commit before Monday's talk, including the PDF of the schematic to make it accessible.
Parts:
- gave numbers to parts that had none: 3
Other:
- note added: "Here, the instruction decoded is implemented using a single 4-bit"
- note added: "The counter is incremented by the system clock, which thus sets the"
- note added: "The instruction decoder, as the name suggests, decodes instructions. It"
- note added: "address (this isn't strictly true, and we could very much optimise this"
- note added: "and probably save an EEPROM, but in the interest of keeping this nice"
- note added: "and understandable, this is how I've done it here - ask me about it if"
- note added: "control signal for that instruction, at that step, depending on the status of"
- note added: "counter 74HC163 chip and two AT28C64B, whic are necessary since"
- note added: "does so by looking up the instruction's 'op-code' (the 4-bit binary"
- note added: "each instruction has at most 8) in an EEPROM. The EEPROMs use"
- note added: "jump if A = B)."
- note added: "operand from the instruction register), and the current step (of which"
- note added: "speed at which the whole computer runs."
- note added: "the comparison unit (which is useful for conditional jump instructions, ie"
- note added: "these two fields, along with the current output status of the comparison"
- note added: "to their address lines, but each one outputs to 8 different control signals."
- note added: "unit as an address, where the data at that address is the value of each"
- note added: "we have 16 control signals and each one can only set 8 for any given"
- note added: "you're interested). Both of the EEPROMS have exactly the same inputs"
- moved on the sheet: U14, U15, U16
