File: kicad/instruction-register.sch (KiCad schematic (older format))
At the start: 2 parts

Commit message: Final Commit Pre-Talk The final commit before Monday's talk, including the PDF of the schematic to make it accessible.
Parts:
- gave numbers to parts that had none: 2
Other:
- note added: "The instruction register is identical to the general purpose registers,"
- note added: "an 'output address to RAM signal'."
- note added: "code to control signals so that they can be executed and it constantly"
- note added: "data bus. It constantly outputs its 4 most significant bits to the"
- note added: "except that it only outputs its 4 least significant bits to the data bus"
- note added: "instruction decoder, for it to decode the instructions from machine"
- note added: "only thing that assets those lines, so it saves control signals to not have"
- note added: "outputs its 4 least significant bits to the RAM's address bus, as it is the"
- note added: "since the others are used for operands which shouldn't ever go on the"
- moved on the sheet: U12, U13
