File: kicad/program-counter.sch (KiCad schematic (older format))
At the start: 2 parts

Commit message: Final Commit Pre-Talk The final commit before Monday's talk, including the PDF of the schematic to make it accessible.
Parts:
- gave numbers to parts that had none: 2
Other:
- note added: "PJ control signal."
- note added: "The program counter is implemented with 2 4-bit counters, which are"
- note added: "The program counter stores the next address within the program"
- note added: "binary counting works (I'll probably demonstrate this more clearly"
- note added: "by 1 with the PI control signal, or set to the value of the data bus with the"
- note added: "outputs connected to the 'count' bus, which goes to the address lines of"
- note added: "program storage."
- note added: "storage to fetch an instruction from. Its count can either be incremented"
- note added: "synchronised through the use of a 'ripple carry' - ie once one reaches"
- note added: "the maximum and resets, it causes the other to count one, which is how"
- note added: "their inputs connected to the data bus and PI/PJ control signals and their"
- note added: "while I'm talking through it). The counters used are 74HC163s, with"
- moved on the sheet: U19, U20
